File: PCB/Platform/Platform.kicad_pcb (KiCad board)
At the start: 2 copper layers, 110 x 100 mm, 20 parts, among them J1 Program, J10 Pin_SERIAL, J2 Conn_01x02_Pin, J3 Conn_01x02_Pin, J4 Pin_LCD_I2C, J5 Pin_RTC, J6 Micro_SD_Card, J8 Pin_SPI_1, J9 Pin_I2C_eksternal, SW1 SW_Push, SW2 SW_Push, U2 MAX485_MODULE_5V_LOGIC_TLL_TO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

Commit message: Update 5 Oktober 2026
Parts:
- removed A2: Clone_Pro_Mini_Socket, PCM_arduino-library:Clone_Pro_Mini_Socket
- removed D1, D2: LED, LED_THT:LED_D5.0mm
- removed J1: Program, Connector_PinSocket_2.54mm:PinSocket_1x06_P2.54mm_Vertical
- removed J10: Pin_SERIAL, Connector_PinHeader_2.54mm:PinHeader_1x04_P2.54mm_Vertical
- removed J2, J3: Conn_01x02_Pin, TerminalBlock_Phoenix:TerminalBlock_Phoenix_MKDS-1,5-2_1x02_P5.00mm_Horizontal
- removed J4: Pin_LCD_I2C, LCD-16X2:MODULE_LCD-16X2
- removed J5: Pin_RTC, DS3231:DS3231
- removed J6: Micro_SD_Card, Connector_PinSocket_2.54mm:PinSocket_1x06_P2.54mm_Vertical
- removed J8: Pin_SPI_1, Connector_PinHeader_2.54mm:PinHeader_1x06_P2.54mm_Vertical
- removed J9: Pin_I2C_eksternal, Connector_PinHeader_2.54mm:PinHeader_1x04_P2.54mm_Vertical
- removed PS1: LM2596, MC00100:CONV_MC00100
- removed R1, R2: 220Ω, Resistor_THT:R_Axial_DIN0207_L6.3mm_D2.5mm_P10.16mm_Horizontal
- removed R3, R4: 1kΩ, Resistor_THT:R_Axial_DIN0207_L6.3mm_D2.5mm_P10.16mm_Horizontal
- removed SW1, SW2: SW_Push, Button_Switch_THT:SW_PUSH_6mm
- removed U2: MAX485_MODULE_5V_LOGIC_TLL_TO_RS-485_CONVERTER, MAX485_MODULE_5V_LOGIC_TLL_TO_RS-485_CONVERTER:MODULE_MAX485_MODULE_5V_LOGIC_TLL_TO_RS-485_CONVERTER
- added ANALOG: Pin_Analog, Connector_PinHeader_2.54mm:PinHeader_1x06_P2.54mm_Vertical, F.Cu at (127.6, 127.2)
- added ARDUINO PRO MINI: Clone_Pro_Mini_Socket, PCM_arduino-library:Clone_Pro_Mini_Socket, F.Cu at (106.3, 87.9)
- added G***: LOGO, LOGO, F.Cu at (85.0, 139.2)
- added I2C: Pin_I2C_eksternal, Connector_PinHeader_2.54mm:PinHeader_1x04_P2.54mm_Vertical, F.Cu at (97.8, 127.2)
- added JP1: SolderJumper_2_Bridged, Jumper:SolderJumper-2_P1.3mm_Bridged_Pad1.0x1.5mm, F.Cu at (61.8, 116.0)
- added JP2: SolderJumper_2_Bridged, Jumper:SolderJumper-2_P1.3mm_Bridged_Pad1.0x1.5mm, F.Cu at (61.8, 120.5)
- added LCD I2C: Pin_LCD_I2C, LCD-16X2:MODULE_LCD-16X2, F.Cu at (130.4, 57.2)
- added LED 1: LED, LED_THT:LED_D5.0mm, F.Cu at (78.2, 118.2)
- added LED 2: LED, LED_THT:LED_D5.0mm, F.Cu at (69.4, 118.2)
- added LM2596: LM2596, MC00100:CONV_MC00100, F.Cu at (73.4, 75.7)
- added POWER INPUT: Conn_01x02_Pin, TerminalBlock_Phoenix:TerminalBlock_Phoenix_MKDS-1,5-2_1x02_P5.00mm_Horizontal, F.Cu at (78.8, 45.0)
- added POWER OUTPUT: Conn_01x02_Pin, TerminalBlock_Phoenix:TerminalBlock_Phoenix_MKDS-1,5-2_1x02_P5.00mm_Horizontal, F.Cu at (64.2, 45.2)
- added PROGRAM: Program, Connector_PinSocket_2.54mm:PinSocket_1x06_P2.54mm_Vertical, F.Cu at (156.6, 127.2)
- added PUSH_BUTTON: SW_Push, Button_Switch_THT:SW_PUSH_6mm, F.Cu at (62.4, 126.7)
- added PUSH_BUTTON: SW_Push, Button_Switch_THT:SW_PUSH_6mm, F.Cu at (73.7, 126.7)
- added REF**: MountingHole_3.2mm_M3, MountingHole:MountingHole_3.2mm_M3, F.Cu at (59.2, 34.2)
- added REF**: MountingHole_3.2mm_M3, MountingHole:MountingHole_3.2mm_M3, F.Cu at (169.8, 139.8)
- added REF**: MountingHole_3.2mm_M3, MountingHole:MountingHole_3.2mm_M3, F.Cu at (59.2, 139.8)
- added REF**: MountingHole_3.2mm_M3, MountingHole:MountingHole_3.2mm_M3, F.Cu at (169.8, 34.2)
- added RESET: RST, Button_Switch_THT:SW_PUSH_6mm, F.Cu at (85.7, 127.0)
- added RS485: MAX485_MODULE_5V_LOGIC_TLL_TO_RS-485_CONVERTER, MAX485_MODULE_5V_LOGIC_TLL_TO_RS-485_CONVERTER:MODULE_MAX485_MODULE_5V_LOGIC_TLL_TO_RS-485_CONVERTER, F.Cu at (148.8, 85.2)
- added RTC DS3231: Pin_RTC, DS3231:DS3231, F.Cu at (103.2, 111.3)
- added R_1K: 1kΩ, Resistor_THT:R_Axial_DIN0207_L6.3mm_D2.5mm_P10.16mm_Horizontal, F.Cu at (74.4, 101.1)
- added R_1K: 1kΩ, Resistor_THT:R_Axial_DIN0207_L6.3mm_D2.5mm_P10.16mm_Horizontal, F.Cu at (79.9, 101.1)
- added R_220: 220Ω, Resistor_THT:R_Axial_DIN0207_L6.3mm_D2.5mm_P10.16mm_Horizontal, F.Cu at (62.4, 101.1)
- added R_220: 220Ω, Resistor_THT:R_Axial_DIN0207_L6.3mm_D2.5mm_P10.16mm_Horizontal, F.Cu at (67.9, 101.1)
- added SDCARD MODULE: Micro_SD_Card, modulsdcard:modul sdcard, F.Cu at (148.8, 109.6)
- added SERIAL: Pin_SERIAL, Connector_PinHeader_2.54mm:PinHeader_1x04_P2.54mm_Vertical, F.Cu at (144.6, 127.2)
- added SPI: Pin_SPI_1, Connector_PinHeader_2.54mm:PinHeader_1x06_P2.54mm_Vertical, F.Cu at (110.3, 127.2)
Routing:
- net +5V: track 0.00 -> 280.7 mm, vias 0 -> 2
- net /I2C_UART_BUS.SDA: track 0.00 -> 95.9 mm, vias 0 -> 1
- net /I2C_UART_BUS.RX: track 0.00 -> 82.3 mm
- net /I2C_UART_BUS.TX: track 0.00 -> 81.2 mm
- net Net-(J1-Pin_3): track 0.00 -> 73.7 mm
- net /SPI_BUS.MOSI: track 0.00 -> 73.4 mm
- net GND: track 0.00 -> 70.2 mm, vias 0 -> 4
- net Net-(A2-RESET-PadRST1): track 0.00 -> 65.9 mm
- net Net-(J1-Pin_2): track 0.00 -> 64.6 mm
- net /RS485_CTRL: track 0.00 -> 64.3 mm
- net Net-(A2-~{DTR}): track 0.00 -> 63.7 mm
- net /A6: track 0.00 -> 58.0 mm
- net Net-(J2-Pin_2): track 0.00 -> 57.5 mm, vias 0 -> 1
- net Net-(J2-Pin_1): track 0.00 -> 56.9 mm
- net /A7: track 0.00 -> 56.6 mm
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- added copper zone on B.Cu, net GND
Other:
- board size 110 x 100 mm -> 123 x 116 mm
- board text added: "5V"
- board text added: "A0"
- board text added: "A1"
- board text added: "A2"
- board text added: "A3"
- board text added: "A6"
- board text added: "A7"
- board text added: "Alicia & Dimas BRIN-2026"
- board text added: "DTR"
- board text added: "GND"
- board text added: "MISO"
- board text added: "MOSI"
- board text added: "RX"
- board text added: "SCK"
- board text added: "SCL"
- board text added: "SDA"
- board text added: "SS"
- board text added: "TX"
- board text added: "VCC"

Commit message: Update 8 Oktober 2026
Parts:
- removed I2C: Pin_I2C_eksternal, Connector_PinHeader_2.54mm:PinHeader_1x04_P2.54mm_Vertical
- added ?: , , F.Cu at (457.9, 38.1)
- added ?: , , F.Cu at (568.4, 38.1)
- added ?: , , F.Cu at (457.9, 143.6)
- added ?: , , F.Cu at (568.4, 143.6)
- added J12: PWR External, Connector_PinHeader_2.54mm:PinHeader_1x03_P2.54mm_Vertical, F.Cu at (126.6, 133.7)
- added J9: Pin_I2C_eksternal, Connector_PinHeader_2.54mm:PinHeader_1x04_P2.54mm_Vertical, F.Cu at (98.0, 127.5)
- added RN1: R_Network09_US, Resistor_THT:R_Array_SIP10, F.Cu at (97.4, 133.9)
- A2: renamed from ARDUINO PRO MINI
- D1: renamed from LED 1
- D2: renamed from LED 2
- J2: renamed from POWER INPUT
- J3: renamed from POWER OUTPUT
- J5: renamed from RTC DS3231
- J6: renamed from SDCARD MODULE
- J7: renamed from LCD I2C; value Pin_LCD_I2C -> Pin_LCD
- renumbered PROGRAM to J1, SERIAL to J10, ANALOG to J4, SPI to J8, LM2596 to PS1, R_220 to R1, R_220 to R2, R_1K to R3, R_1K to R4, PUSH_BUTTON to SW1, PUSH_BUTTON to SW2, RESET to SW3, RS485 to U2
Connections:
- net Net-(A2-RESET-PadRST1) renamed /RST
- net Net-(J2-Pin_1) renamed /V_RAW
- A2 pad RAW: unconnected-(A2-PadRAW) -> +5V
- A2 pad Vcc1: +5V -> +3.3V
- A2 pad Vcc2: unconnected-(A2-Vcc-PadVcc2) -> Net-(J1-Pin_4)
- J1 pad 4: unconnected-(J1-Pin_4-Pad4) -> Net-(J1-Pin_4)
- J5 pad 2: +5V -> +3.3V
- J7 pad 2: +5V -> +3.3V
Routing:
- net +3.3V: track 0.00 -> 174.1 mm
- net Net-(J1-Pin_4): track 0.00 -> 65.4 mm, vias 0 -> 1
- net +5V: track 280.7 -> 294.7 mm
- net /I2C_UART_BUS.SCL: track 50.6 -> 58.6 mm
- net /I2C_UART_BUS.SDA: track 95.9 -> 103.9 mm
- net /RST: track 65.9 -> 62.2 mm
- net GND: track 70.2 -> 73.0 mm
Other:
- board text added: "3.3V"
