File: PCB/Platform/Platform.kicad_sch (KiCad schematic)
At the start: 20 parts, among them J1 Program, J10 Pin_SERIAL, J2 Conn_01x02_Pin, J3 Conn_01x02_Pin, J4 Pin_LCD_I2C, J5 Pin_RTC, J6 Micro_SD_Card, J8 Pin_SPI_1, J9 Pin_I2C_eksternal, SW1 SW_Push, SW2 SW_Push, U2 MAX485_MODULE_5V_LOGIC_TLL_TO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

Commit message: Update 5 Oktober 2026
Parts:
- added J7: Pin_LCD, DS3231:DS3231, symbol Connector:Conn_01x04_Pin
- added JP1, JP2: SolderJumper_2_Bridged, Jumper:SolderJumper-2_P1.3mm_Bridged_Pad1.0x1.5mm, symbol Jumper:SolderJumper_2_Bridged
- added R5: 10kΩ, symbol Device:R
- added R6: 20kΩ, symbol Device:R
- added SW3: RST, Button_Switch_THT:SW_PUSH_6mm, symbol Switch:SW_Push
- added U3: Ai-Thinker-Ra-02, RF_Module:Ai-Thinker-Ra-01-LoRa, symbol RF_Module:Ai-Thinker-Ra-02
- J4: value Pin_LCD_I2C -> Pin_Analog; footprint LCD-16X2:MODULE_LCD-16X2 -> Connector_PinHeader_2.54mm:PinHeader_1x04_P2.54mm_Horizontal
- J6: footprint Connector_PinSocket_2.54mm:PinSocket_1x06_P2.54mm_Vertical -> modulsdcard:modul sdcard
Connections:
- net +5V: now also J7.2 (Pin_2); no longer J4.2 (Pin_2)
- net GND: now also J7.1 (Pin_1), JP1.2 (B), JP2.2 (B), R6.2, SW3.2; no longer D1.1 (K), D2.1 (K), J4.1 (Pin_1)
- net I2C_UART_BUS.SCL: now also J7.4 (Pin_4); no longer J4.4 (Pin_4)
- net I2C_UART_BUS.SDA: now also J7.3 (Pin_3); no longer J4.3 (Pin_3)
- net V_RAW: now reaches J2.1 (Pin_1), PS1.IN+
- net SIM_TX: now reaches A2.A0
- net at A2.A1: now also R5.1
- net A2: now reaches A2.A2
- net A2: now also J4.4 (Pin_4)
- net A3: now reaches A2.A3
- net A3: now also J4.3 (Pin_3)
- net A6: now reaches A2.A6
- net A6: now also J4.2 (Pin_2)
- net A7: now reaches A2.A7
- net A7: now also J4.1 (Pin_1)
- net RST: now reaches A2.RST1 (RESET)
- net RST: now also A2.RST2 (RESET), SW3.1
- new net: D1.1 (K), JP1.1 (A)
- new net: U3.1 (GND), U3.16 (GND), U3.2 (GND), U3.9 (GND)
- new net: D2.1 (K), JP2.1 (A)
- new net SIM_RX: R5.2, R6.1
- no-connect marks 17 -> 9
Other:
- note added: "PLATFORMv1 TRAINER KIT DIMAS_ALICIA"
- note removed: "PLATFORM TRAINER KIT DIMAS_ALICIA"
- moved on the sheet: J10, J5, J9, U2

Commit message: Update 8 Oktober 2026
Parts:
- removed J4: Pin_Analog, Connector_PinHeader_2.54mm:PinHeader_1x04_P2.54mm_Horizontal, symbol Connector:Conn_01x04_Pin
- removed R5: 10kΩ, symbol Device:R
- removed R6: 20kΩ, symbol Device:R
- removed U3: Ai-Thinker-Ra-02, RF_Module:Ai-Thinker-Ra-01-LoRa, symbol RF_Module:Ai-Thinker-Ra-02
- added J12: PWR External, Connector_PinHeader_2.54mm:PinHeader_1x03_P2.54mm_Vertical, symbol Connector:Conn_01x03_Pin
- added J4: Pin_Analog, Connector_PinHeader_2.54mm:PinHeader_1x06_P2.54mm_Vertical, symbol Connector:Conn_01x06_Pin
- added RN1: R_Network09_US, Resistor_THT:R_Array_SIP10, symbol Device:R_Network09_US
- J7: footprint DS3231:DS3231 -> LCD-16X2:MODULE_LCD-16X2
Connections:
- net +5V: now also A2.RAW, J12.3 (Pin_3), RN1.1 (common); no longer A2.Vcc1 (Vcc), J5.2 (Pin_2), J7.2 (Pin_2), J9.2 (Pin_2)
- net A2: now also J4.4 (Pin_4)
- net A3: now also J4.3 (Pin_3)
- net A6: now also J4.2 (Pin_2)
- net A7: now also J4.1 (Pin_1)
- net GND: now also J12.1 (Pin_1)
- net I2C_UART_BUS.SCL: now also RN1.3 (R2)
- net I2C_UART_BUS.SDA: now also RN1.2 (R1)
- net A1: now reaches A2.A1
- net A1: now also J4.5 (Pin_5)
- net at A2.Vcc2 (Vcc): now also J1.4 (Pin_4)
- net SIM_TX renamed A0
- net A0: now also J4.6 (Pin_6)
- new net +3.3V: A2.Vcc1 (Vcc), J12.2 (Pin_2), J5.2 (Pin_2), J7.2 (Pin_2), J9.2 (Pin_2)
- no-connect marks 9 -> 13
Other:
- moved on the sheet: U2
