File: PCB/Platformv2/Platformv2.kicad_sch (KiCad schematic)
At the start: 38 parts, among them J1 Program, J10 Pin_SERIAL, J12 Pin_DIO_LORA, J2 Conn_01x02_Pin, J3 Conn_01x02_Pin, J4 Pin_SIM800L, J5 Pin_RTC, J6 Micro_SD_Card, J7 Pin_Analog, J8 Pin_SPI_1, J9 Pin_I2C_eksternal, SW1 SW_Push, SW2 SW_Push, SW3 RST, U1 SIM800L-CORE, U2 MAX485_MODULE_5V_LOGIC_TLL_TO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, U3 Ai-Thinker-Ra-02, U4 AMS1117CD-3.3

Commit message: Update 8 Oktober 2026
Parts:
- removed J5: Pin_RTC, DS3231:DS3231, symbol Connector:Conn_01x04_Pin
- removed R8, R9: R, symbol Device:R
- removed U3: Ai-Thinker-Ra-02, RF_Module:Ai-Thinker-Ra-01-LoRa, symbol RF_Module:Ai-Thinker-Ra-02
- removed U4: AMS1117CD-3.3, Package_TO_SOT_SMD:TO-252-3_TabPin2, symbol Regulator_Linear:AMS1117CD-3.3
- removed dsn-mini-1: (no value), Mini360_step-down:Mini360_step-down, symbol KICAD_PARTS:dsn-mini-360
- added J11: Pin_RTC, DS3231:DS3231, symbol Connector:Conn_01x06_Pin
- added LORA-RFM-1: (no value), lora_module:lora, symbol LORA:LORA-RFM96
- added RN1: R_Network09_US, Resistor_THT:R_Array_SIP10, symbol Device:R_Network09_US
- added U3: (no value), Mini360_step_down_converter:Untitled, symbol dsn:dsn
Connections:
- net +5V: now also A2.RAW, J6.VCC, J11.VCC (Pin_2), RN1.1 (common); no longer A2.Vcc1 (Vcc), J6.4 (VDD)
- net GND: now also J6.GND, J11.GND (Pin_1), LORA-RFM-1.G, U3.IN-, U3.OUT-; no longer J6.6 (VSS)
- net I2C_UART_BUS.RX: now also RN1.3 (R2)
- net I2C_UART_BUS.SCL: now also J11.SCL (Pin_4)
- net I2C_UART_BUS.SDA: now also J11.SDA (Pin_3)
- net I2C_UART_BUS.TX: now also RN1.2 (R1)
- net LORA_CS: now also LORA-RFM-1.NSS
- net LORA_DIO0: now also LORA-RFM-1.D0
- net LORA_DIO1: now also LORA-RFM-1.D1
- net LORA_DIO2: now also LORA-RFM-1.D2
- net LORA_DIO3: now also LORA-RFM-1.D3
- net LORA_DIO4: now also LORA-RFM-1.D4
- net LORA_DIO5: now also LORA-RFM-1.D5
- net RST: now also LORA-RFM-1.RST
- net SPI_BUS.MISO: now also J6.MISO, LORA-RFM-1.MISO; no longer J6.7 (DAT0)
- net SPI_BUS.MOSI: now also J6.MOSI, LORA-RFM-1.MOSI; no longer J6.3 (CMD)
- net SPI_BUS.SCK: now also J6.SCK, LORA-RFM-1.SCK; no longer J6.5 (CLK)
- net SPI_BUS.SD_CS: now also J6.CS; no longer J6.2 (DAT3/CD)
- net V_RAW: now also U3.IN+
- net at JP3.1 (A): now also U3.OUT+
- new net +3.3V: A2.Vcc1 (Vcc), LORA-RFM-1.3V3
- no-connect marks 9 -> 16
Other:
- moved on the sheet: J12, J6, J7
